Commit message: added rviz

File: galax_bringup/urdf/galax.urdf.xacro (robot description, xacro)
@@ -6,12 +6,12 @@
   <xacro:include filename="$(find urg_node)/urdf/hokuyo_ust10.urdf.xacro"/>
   <!-- Base Link -->
-  <link name="base_link"/>
+  <link name="world"/>
   <!-- Instantiate the Pioneer3DX -->
-  <xacro:pioneer3dx prefix="pioneer3dx_" parent="base_link">
+  <xacro:pioneer3dx prefix="pioneer3dx_" parent="world">
     <origin xyz="0 0 0" rpy="0 0 0"/>
   </xacro:pioneer3dx>
-  <!-- Mount the diffdrive -->
+  <!-- Add the diffdrive controler -->
   <xacro:include filename="$(find diffdrive_arduino)/urdf/diffbot.ros2_control.xacro" />
-  <xacro:diffbot_ros2_control name="DiffBot" prefix="pioneer3dx_" />
+  <xacro:diffbot_ros2_control name="DiffBot" prefix="pioneer3dx_" device="/dev/ttyACM0" baud_rate="57600"/>
   <!-- Mount the lidar -->
   <xacro:hokuyo_ust10_mount prefix="hokuyo_" topic="scan" parent_link="pioneer3dx_top_plate">

Commit message: fixed bringup

File: galax_bringup/urdf/galax.urdf.xacro (robot description, xacro)
@@ -5,8 +5,6 @@
   <!-- Include the Lidar macro -->
   <xacro:include filename="$(find urg_node)/urdf/hokuyo_ust10.urdf.xacro"/>
-  <!-- Base Link -->
-  <link name="world"/>
   <!-- Instantiate the Pioneer3DX -->
-  <xacro:pioneer3dx prefix="pioneer3dx_" parent="world">
+  <xacro:pioneer3dx prefix="pioneer3dx_">
     <origin xyz="0 0 0" rpy="0 0 0"/>
   </xacro:pioneer3dx>
@@ -15,5 +13,5 @@
   <xacro:diffbot_ros2_control name="DiffBot" prefix="pioneer3dx_" device="/dev/ttyACM0" baud_rate="57600"/>
   <!-- Mount the lidar -->
-  <xacro:hokuyo_ust10_mount prefix="hokuyo_" topic="scan" parent_link="pioneer3dx_top_plate">
+  <xacro:hokuyo_ust10_mount prefix="hokuyo" topic="scan" parent_link="pioneer3dx_top_plate">
     <origin xyz="0.16 0 0" rpy="0 0 0"/>
   </xacro:hokuyo_ust10_mount>

Commit message: simulator added

File: galax_bringup/urdf/galax.urdf.xacro (robot description, xacro)
@@ -4,9 +4,22 @@
   <xacro:arg name="use_ros2_control" default="true"/>
   <xacro:arg name="sim_mode" default="false"/>
-  <!-- Instantiate the Pioneer3DX -->
-  <xacro:include filename="$(find amr-ros-config)/urdf/pioneer3dx/pioneer3dx.urdf.xacro"/>
-  <xacro:pioneer3dx prefix="pioneer3dx_">
-    <origin xyz="0 0 0" rpy="0 0 0"/>
-  </xacro:pioneer3dx>
+  <!-- ROBOT -->
+  <!-- Add the real robot -->
+  <xacro:unless value="$(arg sim_mode)">
+    <!-- Instantiate the Pioneer3DX -->
+    <xacro:include filename="$(find amr-ros-config)/urdf/pioneer3dx/pioneer3dx.urdf.xacro"/>
+    <xacro:pioneer3dx prefix="pioneer3dx_">
+      <origin xyz="0 0 0" rpy="0 0 0"/>
+    </xacro:pioneer3dx>
+  </xacro:unless>
+  <!-- Or the simulated robot -->
+  <xacro:if value="$(arg sim_mode)">
+    <!-- Instantiate the Pioneer3DX -->
+    <xacro:include filename="$(find amr-ros-config)/urdf/pioneer3dx/pioneer3dx_sim.urdf.xacro"/>
+    <xacro:pioneer3dx prefix="pioneer3dx_">
+      <origin xyz="0 0 0" rpy="0 0 0"/>
+    </xacro:pioneer3dx>
+  </xacro:if>
+  <!-- CONTROLLER -->
   <!-- Add the diffdrive controler -->
   <xacro:unless value="$(arg sim_mode)">
@@ -19,4 +32,5 @@
     <xacro:pioneer3dx_gazebo_control prefix="pioneer3dx_"/>
   </xacro:if>
+  <!-- LIDAR -->
   <!-- Mount the lidar -->
   <xacro:include filename="$(find urg_node)/urdf/hokuyo_ust10.urdf.xacro"/>

Commit message: fixing robot 2nd attempt

File: galax_bringup/urdf/galax.urdf.xacro (robot description, xacro)
@@ -1,7 +1,7 @@
 <?xml version="1.0"?>
-<robot name="galax" xmlns:xacro="http://ros.org/wiki/xacro">
+<robot xmlns:xacro="http://ros.org/wiki/xacro" name="galax_robot" >
   <!-- Load the arguments -->
   <xacro:arg name="use_ros2_control" default="true"/>
-  <xacro:arg name="sim_mode" default="false"/>
+  <xacro:arg name="sim_mode" default="true"/>
   <!-- ROBOT -->
   <!-- Add the real robot -->

File: galax_description/description/robot.urdf.xacro (robot description, xacro)
@@ -1,44 +1,30 @@
 <?xml version="1.0"?>
 <robot xmlns:xacro="http://ros.org/wiki/xacro" name="galax_robot" >
-  <!-- Load the arguments -->
-  <xacro:arg name="use_ros2_control" default="true"/>
-  <xacro:arg name="sim_mode" default="true"/>
-  <!-- ROBOT -->
-  <!-- Add the real robot -->
-  <xacro:unless value="$(arg sim_mode)">
-    <!-- Instantiate the Pioneer3DX -->
-    <!-- <xacro:include filename="$(find galax_description)/urdf/pioneer3dx/pioneer3dx.urdf.xacro"/>
-    <xacro:pioneer3dx prefix="pioneer3dx_">
-      <origin xyz="0 0 0" rpy="0 0 0"/>
-    </xacro:pioneer3dx> -->
-  </xacro:unless>
-  <!-- Or the simulated robot -->
-  <xacro:if value="$(arg sim_mode)">
-    <!-- Instantiate the Pioneer3DX -->
-    <!-- <xacro:include filename="$(find galax_description)/urdf/pioneer3dx/pioneer3dx_sim.urdf.xacro"/>
-    <xacro:pioneer3dx prefix="pioneer3dx_">
-      	<origin xyz="0 0 0" rpy="0 0 0"/>
-    </xacro:pioneer3dx> -->
-	<xacro:include filename="robot_core.xacro" />
-    <xacro:articubot prefix="pioneer3dx_">
-    	<origin xyz="0 0 0" rpy="0 0 0"/>
-    </xacro:articubot>
-  </xacro:if>
+	<!-- Load the arguments -->
+	<xacro:arg name="use_ros2_control" default="true"/>
+	<xacro:arg name="sim_mode" default="true"/>
+	<!-- ROBOT -->
+	<!-- Add the real robot -->
+	<xacro:unless value="$(arg sim_mode)">
+		<!-- Instantiate the Pioneer3DX -->
+	</xacro:unless>
+	<!-- Or the simulated robot -->
+	<xacro:if value="$(arg sim_mode)">
+		<!-- Instantiate the Pioneer3DX -->
+		<xacro:include filename="$(find galax_description)/description/robot_core.xacro"/>
+		<xacro:pioneer3dx prefix="">
+			<origin xyz="0 0 0" rpy="0 0 0"/>
+		</xacro:pioneer3dx>
+	</xacro:if>
   <!-- CONTROLLER -->
   <!-- Add the diffdrive controler -->
   <xacro:unless value="$(arg sim_mode)">
-		<xacro:include filename="$(find diffdrive_arduino)/urdf/diffbot.ros2_control.xacro" />
-		<xacro:diffbot_ros2_control name="DiffBot" prefix="pioneer3dx_" device="/dev/ttyACM0" baud_rate="57600"/>
+    <xacro:include filename="$(find diffdrive_arduino)/urdf/diffbot.ros2_control.xacro" />
+    <xacro:diffbot_ros2_control name="DiffBot" prefix="pioneer3dx_" device="/dev/ttyACM0" baud_rate="57600"/>
   </xacro:unless>
   <!-- Or the Gazebo plugin -->
   <xacro:if value="$(arg sim_mode)">
-		<xacro:include filename="$(find galax_description)/urdf/gazebo_control.xacro"/>
-		<xacro:pioneer3dx_gazebo_control prefix=""/>
+    <xacro:include filename="$(find galax_description)/urdf/gazebo_control.xacro"/>
+    <xacro:gazebo_control prefix=""/>
   </xacro:if>
-  <!-- LIDAR -->
-  <!-- Mount the lidar -->
-  <!-- <xacro:include filename="$(find urg_node)/urdf/hokuyo_ust10.urdf.xacro"/>
-  <xacro:hokuyo_ust10_mount prefix="hokuyo" topic="scan" parent_link="chasis">
-		<origin xyz="0.16 0 0" rpy="0 0 0"/>
-  </xacro:hokuyo_ust10_mount> -->
 </robot>
