Commit message: fixing robot 3rd attempt

File: galax_description/description/gazebo_control.xacro (robot description, xacro)
@@ -1,21 +1,32 @@
 <?xml version="1.0"?>
-<robot xmlns:xacro="http://www.ros.org/wiki/xacro">
-    <gazebo>
-        <plugin name="diff_drive" filename="libgazebo_ros_diff_drive.so">
-            <!-- Wheel Information -->
-            <left_joint>left_wheel_joint</left_joint>
-            <right_joint>right_wheel_joint</right_joint>
-            <wheel_separation>0.297</wheel_separation>
-            <wheel_diameter>0.066</wheel_diameter>
-            <!-- Limits -->
-            <max_wheel_torque>200</max_wheel_torque>
-            <max_wheel_acceleration>10.0</max_wheel_acceleration>
-            <!-- Output -->
-            <odometry_frame>odom</odometry_frame>
-            <robot_base_frame>base_link</robot_base_frame>
-            <publish_odom>true</publish_odom>
-            <publish_odom_tf>true</publish_odom_tf>
-            <publish_wheel_tf>true</publish_wheel_tf>
-        </plugin>
-    </gazebo>
+<robot xmlns:xacro="http://ros.org/wiki/xacro">
+    <xacro:macro name="pioneer3dx_gazebo_control" params="prefix">
+        <ros2_control name="GazeboSystem" type="system">
+            <hardware>
+                <plugin>gazebo_ros2_control/GazeboSystem</plugin>
+            </hardware>
+            <joint name="${prefix}left_wheel_joint">
+                <command_interface name="velocity">
+                    <param name="min">-10</param>
+                    <param name="max">10</param>
+                </command_interface>
+                <state_interface name="velocity"/>
+                <state_interface name="position"/>
+            </joint>
+            <joint name="${prefix}right_wheel_joint">
+                <command_interface name="velocity">
+                    <param name="min">-10</param>
+                    <param name="max">10</param>
+                </command_interface>
+                <state_interface name="velocity"/>
+                <state_interface name="position"/>
+            </joint>
+        </ros2_control>
+        <gazebo>
+            <plugin name="gazebo_ros2_control" filename="libgazebo_ros2_control.so">
+                <parameters>$(find galax_description)/config/my_controllers.yaml</parameters>
+				<parameters>$(find galax_description)/config/gaz_ros2_ctl_use_sim.yaml</parameters>
+            </plugin>
+        </gazebo>
+    </xacro:macro>
 </robot>

File: galax_description/description/robot_core.xacro (robot description, xacro)
@@ -1,152 +1,296 @@
 <?xml version="1.0"?>
 <robot xmlns:xacro="http://www.ros.org/wiki/xacro" >
-    <xacro:include filename="inertial_macros.xacro"/>
-    <xacro:macro name="articubot" params="prefix *origin">
-        <xacro:property name="chassis_length" value="0.335"/>
-        <xacro:property name="chassis_width" value="0.265"/>
-        <xacro:property name="chassis_height" value="0.138"/>
-        <xacro:property name="chassis_mass" value="1.0"/>
-        <xacro:property name="wheel_radius" value="0.033"/>
-        <xacro:property name="wheel_thickness" value="0.026"/>
-        <xacro:property name="wheel_mass" value="0.05"/>
-        <xacro:property name="wheel_offset_x" value="0.226"/>
-        <xacro:property name="wheel_offset_y" value="0.1485"/>
-        <xacro:property name="wheel_offset_z" value="0.01"/>
-        <xacro:property name="caster_wheel_radius" value="0.01"/>
-        <xacro:property name="caster_wheel_mass" value="0.01"/>
-        <xacro:property name="caster_wheel_offset_x" value="0.075"/>
-        <xacro:property name="caster_wheel_offset_z" value="${wheel_offset_z - wheel_radius + caster_wheel_radius}"/>
-        <material name="white">
-            <color rgba="1 1 1 1" />
-        </material>
-        <material name="orange">
-            <color rgba="1 0.3 0.1 1"/>
-        </material>
-        <material name="blue">
-            <color rgba="0.2 0.2 1 1"/>
-        </material>
-        <material name="black">
-            <color rgba="0 0 0 1"/>
-        </material>
-        <material name="red">
-            <color rgba="1 0 0 1"/>
-        </material>
+    <xacro:include filename="$(find galax_description)/urdf/materials.xacro"/>
+	<xacro:include filename="$(find galax_description)/urdf/inertial_macros.xacro"/>
+    <xacro:macro name="pioneer3dx" params="prefix *origin">
+		<!-- Chassis -->
+		<xacro:property name="chassis_length" value="0.41"/>
+		<xacro:property name="chassis_width" value="0.272"/>
+		<xacro:property name="chassis_height" value="0.172"/>
+		<xacro:property name="chassis_mass" value="1.0"/>
+		<!-- Top Plate -->
+		<xacro:property name="top_plate_length" value="0.41"/>
+		<xacro:property name="top_plate_width" value="0.272"/>
+		<xacro:property name="top_plate_height" value="0.0052"/>
+		<xacro:property name="top_plate_mass" value="0.01"/>
+		<!-- Wheels -->
+		<xacro:property name="wheel_radius" value="0.09"/>
+		<xacro:property name="wheel_thickness" value="0.04"/>
+		<xacro:property name="wheel_mass" value="0.05"/>
+		<!-- Caster wheel -->
+		<xacro:property name="caster_wheel_radius" value="0.0375"/>
+		<xacro:property name="caster_wheel_thickness" value="0.01"/>
+		<xacro:property name="caster_wheel_mass" value="0.01"/>
         <!-- BASE LINK -->
-        <link name="base_link">
-        </link>
-        <!-- BASE_FOOTPRINT LINK -->
-        <joint name="base_footprint_joint" type="fixed">
-            <parent link="base_link"/>
-            <child link="base_footprint"/>
-            <origin xyz="0 0 0" rpy="0 0 0"/>
-        </joint>
-        <link name="base_footprint">
+        <link name="${prefix}base_link">
         </link>
         <!-- CHASSIS LINK -->
-        <joint name="chassis_joint" type="fixed">
-            <parent link="base_link"/>
-            <child link="chassis"/>
-            <origin xyz="${-wheel_offset_x} 0 ${-wheel_offset_z}"/>
-        </joint>
-        <link name="chassis">
-            <visual>
-                <origin xyz="${chassis_length/2} 0 ${chassis_height/2}"/>
-                <geometry>
-                    <box size="${chassis_length} ${chassis_width} ${chassis_height}"/>
-                </geometry>
-                <material name="orange"/>
-            </visual>
-            <collision>
-                <origin xyz="${chassis_length/2} 0 ${chassis_height/2}"/>
-                <geometry>
-                    <box size="${chassis_length} ${chassis_width} ${chassis_height}"/>
-                </geometry>
-            </collision>
-            <xacro:inertial_box mass="0.5" x="${chassis_length}" y="${chassis_width}" z="${chassis_height}">
-                <origin xyz="${chassis_length/2} 0 ${chassis_height/2}" rpy="0 0 0"/>
-            </xacro:inertial_box>
-        </link>
-        <gazebo reference="chassis">
-            <material>Gazebo/Orange</material>
-        </gazebo>
+		<link name="${prefix}chassis">
+			<visual>
+				<origin xyz="-0.045 0 0.148" rpy="0 0 0"/>
+				<geometry>
+					<mesh filename="file://$(find galax_description)/meshes/chassis.stl"/>
+				</geometry>
+				<material name="ChassisRed"/>
+			</visual>
+			<xacro:inertial_box mass="${chassis_mass}" x="${chassis_length}" y="${chassis_width}" z="${chassis_height}">
+            	<origin xyz="0 0 ${chassis_height/2}" rpy="0 0 0"/>
+        	</xacro:inertial_box>
+		</link>
+		<gazebo reference="${prefix}chassis">
+			<material>Gazebo/Red</material>
+		</gazebo>
+		<joint name="${prefix}chassis_joint" type="fixed">
+			<origin xyz="0 0 0" rpy="0 0 0"/>
+			<parent link="${prefix}base_link"/>
+			<child link="${prefix}chassis"/>
+		</joint>
+		<!-- Top Plate -->
+		<link name="${prefix}top_plate">
+			<visual>
+				<origin xyz="0 0 0" rpy="0 0 0"/>
+				<geometry>
+					<mesh filename="file://$(find galax_description)/meshes/top.stl"/>
+				</geometry>
+				<material name="TopBlack"/>
+			</visual>
+			<xacro:inertial_box mass="${top_plate_mass}" x="${top_plate_length}" y="${top_plate_width}" z="${top_plate_height}">
+            	<origin xyz="0.045 0 ${top_plate_height/2}" rpy="0 0 0"/>
+        	</xacro:inertial_box>
+		</link>
+		<gazebo reference="${prefix}top_plate">
+			<material>Gazebo/Black</material>
+		</gazebo>
+		<joint name="${prefix}base_top_joint" type="fixed">
+			<origin xyz="-0.045 0 0.234" rpy="0 0 0"/>
+			<parent link="${prefix}chassis"/>
+			<child link="${prefix}top_plate"/>
+		</joint>
+		<!-- Front Sonar -->
+		<link name="${prefix}front_sonar">
+			<visual>
+				<origin xyz="0 0 0" rpy="0 0 0"/>
+				<geometry>
+					<mesh filename="file://$(find galax_description)/meshes/front_sonar.stl"/>
+				</geometry>
+				<material name="SonarYellow"/>
+			</visual>
+			<inertial>
+				<mass value="0.0001"/>
+				<origin xyz="0 0 0"/>
+				<inertia ixx="1" ixy="0" ixz="0" iyy="1" iyz="0" izz="1"/>
+			</inertial>
+		</link>
+		<gazebo reference="${prefix}front_sonar">
+			<material value="Gazebo/Yellow"/>
+		</gazebo>
+		<joint name="${prefix}base_front_joint" type="fixed">
+			<origin xyz="-0.198 0 0.208" rpy="0 0 0"/>
+			<parent link="${prefix}chassis"/>
+			<child link="${prefix}front_sonar"/>
+		</joint>
+		<!-- Back Sonar -->
+		<link name="${prefix}back_sonar">
+			<visual>
+				<origin xyz="0 0 0" rpy="0 0 0"/>
+				<geometry>
+					<mesh filename="file://$(find galax_description)/meshes/back_sonar.stl"/>
+				</geometry>
+				<material name="SonarYellow"/>
+			</visual>
+			<inertial>
+				<mass value="0.0001"/>
+				<origin xyz="0 0 0"/>
+				<inertia ixx="1" ixy="0" ixz="0" iyy="1" iyz="0" izz="1"/>
+			</inertial>
+		</link>
+		<gazebo reference="${prefix}back_sonar">
+			<material value="Gazebo/Yellow"/>
+		</gazebo>
+		<joint name="${prefix}base_back_joint" type="fixed">
+			<origin xyz="0.109 0 0.209" rpy="0 0 0"/>
+			<parent link="${prefix}chassis"/>
+			<child link="${prefix}back_sonar"/>
+		</joint>
         <!-- LEFT WHEEL LINK -->
-        <joint name="left_wheel_joint" type="continuous">
-            <parent link="base_link"/>
-            <child link="left_wheel"/>
-            <origin xyz="0 ${wheel_offset_y} 0" rpy="-${pi/2} 0 0" />
-            <axis xyz="0 0 1"/>
-        </joint>
-        <link name="left_wheel">
-            <visual>
-                <geometry>
-                    <cylinder radius="${wheel_radius}" length="${wheel_thickness}"/>
-                </geometry>
-                <material name="blue"/>
-            </visual>
-            <collision>
-                <geometry>
-                    <sphere radius="${wheel_radius}"/>
-                </geometry>
-            </collision>
-            <xacro:inertial_cylinder mass="${wheel_mass}" length="${wheel_thickness}" radius="${wheel_radius}">
-                <origin xyz="0 0 0" rpy="0 0 0"/>
-            </xacro:inertial_cylinder>
-        </link>
-        <gazebo reference="left_wheel">
-            <material>Gazebo/Blue</material>
-        </gazebo>
+		<link name="${prefix}left_hub">
+			<visual>
+				<origin xyz="0 0 0" rpy="${-3.1415927/2.0} 0 0"/>
+				<geometry>
+					<cylinder radius="0.09" length="0.01"/>
+				</geometry>
+				<material name="HubcapYellow"/>
+			</visual>
+			<xacro:inertial_cylinder mass="0.001" length="0.01" radius="0.0375">
+				<origin xyz="0 0 0" rpy="${-3.1415927/2.0} 0 0"/>
+			</xacro:inertial_cylinder>
+		</link>
+		<gazebo reference="${prefix}left_hub">
+			<material value="Gazebo/Yellow"/>
+		</gazebo>
+		<joint name="${prefix}left_hub_joint" type="fixed">
+			<origin xyz="0 0.15 0.08" rpy="0 0 0"/>
+			<parent link="${prefix}chassis"/>
+			<child link="${prefix}left_hub"/>
+			<axis xyz="0 1 0"/>
+		</joint>
+		<link name="${prefix}left_wheel">
+			<collision>
+				<origin xyz="0 0 0" rpy="0 0 0"/>
+				<geometry>
+					<sphere radius="${wheel_radius}"/>
+				</geometry>
+			</collision>
+			<visual>
+				<origin xyz="0 0 0" rpy="1.5708 0 0"/>
+				<geometry>
+					<mesh filename="file://$(find galax_description)/meshes/left_wheel.stl"/>
+				</geometry>
+				<material name="WheelBlack"/>
+			</visual>
+			<xacro:inertial_cylinder mass="${wheel_mass}" length="${wheel_thickness}" radius="${wheel_radius}">
+				<origin xyz="0 0 0" rpy="0 0 0"/>
+			</xacro:inertial_cylinder>
+		</link>
+		<gazebo reference="${prefix}left_wheel">
+			<material value="Gazebo/Black"/>
+            <mu1 value="10000.0"/>
+			<mu2 value="10000.0"/>
+		</gazebo>
+		<joint name="${prefix}left_wheel_joint" type="continuous">
+			<origin xyz="0 0 0" rpy="-1.5708 0 0"/>
+			<axis xyz="0 0 1"/>
+			<parent link="${prefix}left_hub"/>
+			<child link="${prefix}left_wheel"/>
+		</joint>
         <!-- RIGHT WHEEL LINK -->
-        <joint name="right_wheel_joint" type="continuous">
-            <parent link="base_link"/>
-            <child link="right_wheel"/>
-            <origin xyz="0 ${-wheel_offset_y} 0" rpy="${pi/2} 0 0" />
-            <axis xyz="0 0 -1"/>
-        </joint>
-        <link name="right_wheel">
-            <visual>
-                <geometry>
-                    <cylinder radius="${wheel_radius}" length="${wheel_thickness}"/>
-                </geometry>
-                <material name="blue"/>
-            </visual>
-            <collision>
-                <geometry>
-                    <sphere radius="${wheel_radius}"/>
-                </geometry>
-            </collision>
-            <xacro:inertial_cylinder mass="${wheel_mass}" length="${wheel_thickness}" radius="${wheel_radius}">
-                <origin xyz="0 0 0" rpy="0 0 0"/>
-            </xacro:inertial_cylinder>
-        </link>
-        <gazebo reference="right_wheel">
-            <material>Gazebo/Blue</material>
-        </gazebo>
+		<link name="${prefix}right_hub">
+			<visual>
+				<origin xyz="0 0 0" rpy="${3.1415927/2.0} 0 0"/>
+				<geometry>
+					<cylinder radius="0.09" length="0.01"/>
+				</geometry>
+				<material name="HubcapYellow"/>
+			</visual>
+			<xacro:inertial_cylinder mass="0.001" length="0.01" radius="0.0375">
+				<origin xyz="0 0 0" rpy="${3.1415927/2.0} 0 0"/>
+			</xacro:inertial_cylinder>
+		</link>
+		<gazebo reference="${prefix}right_hub">
+			<material value="Gazebo/Yellow"/>
+		</gazebo>
+		<joint name="${prefix}right_hub_joint" type="fixed">
+			<origin xyz="0 -0.15 0.08" rpy="0 0 0"/>
+			<parent link="${prefix}chassis"/>
+			<child link="${prefix}right_hub"/>
+		</joint>
+		<link name="${prefix}right_wheel">
+			<collision>
+				<origin xyz="0 0 0" rpy="0 0 0"/>
+				<geometry>
+					<sphere radius="${wheel_radius}"/>
+				</geometry>
+			</collision>
+			<visual>
+				<origin xyz="0 0 0" rpy="-1.5708 0 0"/>
+				<geometry>
+					<mesh filename="file://$(find galax_description)/meshes/right_wheel.stl"/>
+				</geometry>
+				<material name="WheelBlack"/>
+			</visual>
+			<xacro:inertial_cylinder mass="${wheel_mass}" length="${wheel_thickness}" radius="${wheel_radius}">
+				<origin xyz="0 0 0" rpy="0 0 0"/>
+			</xacro:inertial_cylinder>
+		</link>
+		<gazebo reference="${prefix}right_wheel">
+			<material value="Gazebo/Black"/>
+            <mu1 value="10000000.0"/>
+			<mu2 value="10000000.0"/>
+		</gazebo>
+		<joint name="${prefix}right_wheel_joint" type="continuous">
+			<origin xyz="0 -0.15 0.08" rpy="1.5708 0 0"/>
+			<axis xyz="0 0 -1"/>
+			<parent link="${prefix}chassis"/>
+			<child link="${prefix}right_wheel"/>
+		</joint>
         <!-- CASTER WHEEL LINK -->
-        <joint name="caster_wheel_joint" type="fixed">
-            <parent link="chassis"/>
-            <child link="caster_wheel"/>
-            <origin xyz="${caster_wheel_offset_x} 0 ${caster_wheel_offset_z}"/>
-        </joint>
-        <link name="caster_wheel">
-            <visual>
-                <geometry>
-                    <sphere radius="${caster_wheel_radius}"/>
-                </geometry>
-                <material name="white"/>
-            </visual>
-            <collision>
-                <geometry>
-                    <sphere radius="${caster_wheel_radius}"/>
-                </geometry>
-            </collision>
-            <xacro:inertial_sphere mass="${caster_wheel_mass}" radius="${caster_wheel_radius}">
-                <origin xyz="0 0 0" rpy="0 0 0"/>
-            </xacro:inertial_sphere>
-        </link>
-        <gazebo reference="caster_wheel">
-            <material>Gazebo/White</material>
-            <mu1 value="0.001"/>
-            <mu2 value="0.001"/>
-        </gazebo>
+		<link name="${prefix}caster_swivel">
+			<visual>
+				<origin xyz="0 0 0" rpy="0 0 0"/>
+				<geometry>
+					<mesh filename="file://$(find galax_description)/meshes/caster_swivel.stl"/>
+				</geometry>
+				<material name="ChassisGrey"/>
+			</visual>
+			<inertial>
+				<mass value="0.01"/>
+				<origin xyz="0 0 0"/>
+				<inertia ixx="0.01" ixy="0" ixz="0" iyy="0.01" iyz="0" izz="0.01"/>
+			</inertial>
+		</link>
+		<gazebo reference="${prefix}caster_swivel">
+			<material value="Gazebo/Grey"/>
+		</gazebo>
+		<joint name="${prefix}base_caster_swivel_joint" type="fixed"> <!--Not fixed. Change for simulation -->
+			<origin xyz="-0.185 0 0.045" rpy="0 0 0"/>
+			<axis xyz="0 0 1"/>
+			<parent link="${prefix}chassis"/>
+			<child link="${prefix}caster_swivel"/>
+		</joint>
+		<!-- Hubcap -->
+		<link name="${prefix}caster_hubcap">
+			<visual>
+				<origin xyz="0 0 0" rpy="${1.5708} 0 0"/>
+				<geometry>
+					<mesh filename="file://$(find galax_description)/meshes/caster_hubcap.stl"/>
+				</geometry>
+				<material name="ChassisGrey"/>
+			</visual>
+			<inertial>
+				<mass value="0.01"/>
+				<origin xyz="0 0 0"/>
+				<inertia ixx="0.012411765597" ixy="-0.000711733678" ixz="0.00050272983"
+							iyy="0.015218160428" iyz="-0.000004273467" izz="0.011763977943"/>
+			</inertial>
+		</link>
+		<gazebo reference="${prefix}caster_hubcap">
+			<material value="Gazebo/Grey"/>
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
File: galax_description/urdf/galax.urdf.xacro (robot description, xacro)
@@ -8,6 +8,6 @@
   <xacro:unless value="$(arg sim_mode)">
     <!-- Instantiate the Pioneer3DX -->
-    <xacro:include filename="$(find galax_description)/urdf/pioneer3dx/pioneer3dx.urdf.xacro"/>
-    <xacro:pioneer3dx prefix="pioneer3dx_">
+    <xacro:include filename="$(find galax_description)/urdf/pioneer3dx.urdf.xacro"/>
+    <xacro:pioneer3dx prefix="">
       <origin xyz="0 0 0" rpy="0 0 0"/>
     </xacro:pioneer3dx>
@@ -16,6 +16,6 @@
   <xacro:if value="$(arg sim_mode)">
     <!-- Instantiate the Pioneer3DX -->
-    <xacro:include filename="$(find galax_description)/urdf/pioneer3dx/pioneer3dx_sim.urdf.xacro"/>
-    <xacro:pioneer3dx prefix="pioneer3dx_">
+    <xacro:include filename="$(find galax_description)/urdf/pioneer3dx_sim.urdf.xacro"/>
+    <xacro:pioneer3dx prefix="">
       <origin xyz="0 0 0" rpy="0 0 0"/>
     </xacro:pioneer3dx>
@@ -25,21 +25,16 @@
   <xacro:unless value="$(arg sim_mode)">
     <xacro:include filename="$(find diffdrive_arduino)/urdf/diffbot.ros2_control.xacro" />
-    <xacro:diffbot_ros2_control name="DiffBot" prefix="pioneer3dx_" device="/dev/ttyACM0" baud_rate="57600"/>
+    <xacro:diffbot_ros2_control name="DiffBot" prefix="" device="/dev/ttyACM0" baud_rate="57600"/>
   </xacro:unless>
   <!-- Or the Gazebo plugin -->
   <xacro:if value="$(arg sim_mode)">
-    <xacro:include filename="$(find galax_description)/urdf/pioneer3dx/gazebo_control.xacro"/>
-    <xacro:pioneer3dx_gazebo_control prefix="pioneer3dx_"/>
+    <xacro:include filename="$(find galax_description)/urdf/gazebo_control.xacro"/>
+    <xacro:gazebo_control prefix=""/>
   </xacro:if>
   <!-- LIDAR -->
   <!-- Mount the lidar -->
   <xacro:include filename="$(find urg_node)/urdf/hokuyo_ust10.urdf.xacro"/>
-  <xacro:hokuyo_ust10_mount prefix="hokuyo" topic="scan" parent_link="pioneer3dx_top_plate">
+  <xacro:hokuyo_ust10_mount prefix="hokuyo" topic="scan" parent_link="top_plate">
     <origin xyz="0.16 0 0" rpy="0 0 0"/>
   </xacro:hokuyo_ust10_mount>
-  <!-- COLLISION DETECTOR -->
-  <!-- <xacro:if value="$(arg sim_mode)">
-    <xacro:include filename="$(find galax_description)/urdf/pioneer3dx/gazebo_contact.xacro"/>
-    <xacro:pioneer3dx_collision_controller prefix="pioneer3dx_" link_name="base_link"/>
-  </xacro:if> -->
 </robot>

File: galax_description/urdf/gazebo_control.xacro (robot description, xacro)
@@ -1,23 +1,5 @@
 <?xml version="1.0"?>
 <robot xmlns:xacro="http://ros.org/wiki/xacro">
-    <xacro:macro name="pioneer3dx_gazebo_control" params="prefix">
-        <gazebo>
-            <plugin name="diff_drive" filename="libgazebo_ros_diff_drive.so">
-                <!-- Wheel Information -->
-                <left_joint>${prefix}left_wheel_joint</left_joint>
-                <right_joint>${prefix}right_wheel_joint</right_joint>
-                <wheel_separation>0.30</wheel_separation>
-                <wheel_diameter>0.18</wheel_diameter>
-                <!-- Limits -->
-                <max_wheel_torque>200</max_wheel_torque>
-                <max_wheel_acceleration>10.0</max_wheel_acceleration>
-                <!-- Output -->
-                <odometry_frame>${prefix}odom</odometry_frame>
-                <robot_base_frame>${prefix}base_link</robot_base_frame>
-                <publish_odom>true</publish_odom>
-                <publish_odom_tf>true</publish_odom_tf>
-                <publish_wheel_tf>true</publish_wheel_tf>
-            </plugin>
-        </gazebo>
+    <xacro:macro name="gazebo_control" params="prefix">
         <ros2_control name="GazeboSystem" type="system">
             <hardware>
@@ -43,6 +25,6 @@
         <gazebo>
             <plugin name="gazebo_ros2_control" filename="libgazebo_ros2_control.so">
-                <parameters>$(find amr-ros-config)/config/controller_config.yaml</parameters>
-				<parameters>$(find amr-ros-config)/config/gaz_ros2_ctl_use_sim.yaml</parameters>
+                <parameters>$(find galax_description)/config/my_controllers.yaml</parameters>
+				<parameters>$(find galax_description)/config/gaz_ros2_ctl_use_sim.yaml</parameters>
             </plugin>
         </gazebo>
