Commit message: erased inertias

File: galax_description/urdf/pioneer3dx_sim.urdf.xacro (robot description, xacro)
@@ -30,5 +30,6 @@
 				<origin xyz="${chassis_length/2} 0 ${chassis_height/2}"/>
 				<geometry>
-					<box size="${chassis_length} ${chassis_width} ${chassis_height}"/>
+					<box size="0 0 0"/>
+					<!-- <box size="${chassis_length/4} ${chassis_width/4} ${chassis_height/4}"/> -->
 				</geometry>
 			</collision>
@@ -61,7 +62,4 @@
 				<material name="TopBlack"/>
 			</visual>
-			<xacro:inertial_box mass="${top_plate_mass}" x="${top_plate_length}" y="${top_plate_width}" z="${top_plate_height}">
-            	<origin xyz="0.045 0 ${top_plate_height/2}" rpy="0 0 0"/>
-        	</xacro:inertial_box>
 		</link>
 		<gazebo reference="${prefix}top_plate">
@@ -82,9 +80,4 @@
 				<material name="SonarYellow"/>
 			</visual>
-			<inertial>
-				<mass value="0.0001"/>
-				<origin xyz="0 0 0"/>
-				<inertia ixx="1" ixy="0" ixz="0" iyy="1" iyz="0" izz="1"/>
-			</inertial>
 		</link>
 		<gazebo reference="${prefix}front_sonar">
@@ -105,9 +98,4 @@
 				<material name="SonarYellow"/>
 			</visual>
-			<inertial>
-				<mass value="0.0001"/>
-				<origin xyz="0 0 0"/>
-				<inertia ixx="1" ixy="0" ixz="0" iyy="1" iyz="0" izz="1"/>
-			</inertial>
 		</link>
 		<gazebo reference="${prefix}back_sonar">
@@ -128,7 +116,4 @@
 				<material name="HubcapYellow"/>
 			</visual>
-			<xacro:inertial_cylinder mass="0.001" length="0.01" radius="0.0375">
-				<origin xyz="0 0 0" rpy="${-3.1415927/2.0} 0 0"/>
-			</xacro:inertial_cylinder>
 		</link>
 		<gazebo reference="${prefix}left_hub">
@@ -165,7 +150,7 @@
 		</gazebo>
 		<joint name="${prefix}left_wheel_joint" type="continuous">
-			<origin xyz="0 0 0" rpy="-1.5708 0 0"/>
-			<axis xyz="0 0 1"/>
-			<parent link="${prefix}left_hub"/>
+			<origin xyz="0 0.15 0.08" rpy="-1.5708 0 0"/>
+			<axis xyz="0 0 1"/>
+			<parent link="${prefix}chassis"/>
 			<child link="${prefix}left_wheel"/>
 		</joint>
@@ -179,7 +164,4 @@
 				<material name="HubcapYellow"/>
 			</visual>
-			<xacro:inertial_cylinder mass="0.001" length="0.01" radius="0.0375">
-				<origin xyz="0 0 0" rpy="${3.1415927/2.0} 0 0"/>
-			</xacro:inertial_cylinder>
 		</link>
 		<gazebo reference="${prefix}right_hub">
@@ -229,9 +211,4 @@
 				<material name="ChassisGrey"/>
 			</visual>
-			<inertial>
-				<mass value="0.01"/>
-				<origin xyz="0 0 0"/>
-				<inertia ixx="0.01" ixy="0" ixz="0" iyy="0.01" iyz="0" izz="0.01"/>
-			</inertial>
 		</link>
 		<gazebo reference="${prefix}caster_swivel">
@@ -253,10 +230,4 @@
 				<material name="ChassisGrey"/>
 			</visual>
-			<inertial>
-				<mass value="0.01"/>
-				<origin xyz="0 0 0"/>
-				<inertia ixx="0.012411765597" ixy="-0.000711733678" ixz="0.00050272983"
-							iyy="0.015218160428" iyz="-0.000004273467" izz="0.011763977943"/>
-			</inertial>
 		</link>
 		<gazebo reference="${prefix}caster_hubcap">
@@ -294,7 +265,7 @@
 		</gazebo>
 		<joint name="${prefix}caster_wheel_joint" type="fixed">  <!--Not fixed. Change for simulation -->
-			<origin xyz="-0.0035 0 -0.001" rpy="0 0 0"/>
-			<axis xyz="0 0 1"/>
-			<parent link="${prefix}caster_hubcap"/>
+			<origin xyz="-0.2105 0 0.029" rpy="1.5708 0 0"/>
+			<axis xyz="0 0 1"/>
+			<parent link="${prefix}chassis"/>
 			<child link="${prefix}caster_wheel"/>
 		</joint>

Commit message: missing super power correction+

File: galax_description/urdf/pioneer3dx_sim.urdf.xacro (robot description, xacro)
@@ -8,5 +8,5 @@
 		<xacro:property name="chassis_width" value="0.272"/>
 		<xacro:property name="chassis_height" value="0.172"/>
-		<xacro:property name="chassis_mass" value="1.0"/>
+		<xacro:property name="chassis_mass" value="5.0"/>
 		<!-- Top Plate -->
 		<xacro:property name="top_plate_length" value="0.41"/>
@@ -17,5 +17,5 @@
 		<xacro:property name="wheel_radius" value="0.09"/>
 		<xacro:property name="wheel_thickness" value="0.04"/>
-		<xacro:property name="wheel_mass" value="0.05"/>
+		<xacro:property name="wheel_mass" value="0.5"/>
 		<!-- Caster wheel -->
 		<xacro:property name="caster_wheel_radius" value="0.0375"/>
@@ -28,8 +28,8 @@
 		<link name="${prefix}chassis">
 			<collision>
-				<origin xyz="${chassis_length/2} 0 ${chassis_height/2}"/>
-				<geometry>
-					<box size="0 0 0"/>
-					<!-- <box size="${chassis_length/4} ${chassis_width/4} ${chassis_height/4}"/> -->
+				<origin xyz="0 0 ${chassis_height/2}"/>
+				<geometry>
+					<!-- <box size="0 0 0"/> -->
+					<box size="${chassis_length/4} ${chassis_width/4} ${chassis_height/4}"/>
 				</geometry>
 			</collision>
@@ -270,4 +270,24 @@
 			<child link="${prefix}caster_wheel"/>
 		</joint>
+		<!-- Passive Caster Wheel -->
+		<link name="${prefix}passive_caster_wheel">
+			<collision>
+				<origin xyz="0 0 0" rpy="0 0 0"/>
+				<geometry>
+					<sphere radius="${caster_wheel_radius}"/>
+				</geometry>
+			</collision>
+		</link>
+		<gazebo reference="${prefix}passive_caster_wheel">
+			<material value="Gazebo/White"/>
+			<mu1 value="0.00001"/>
+			<mu2 value="0.00001"/>
+		</gazebo>
+		<joint name="${prefix}passive_caster_wheel_joint" type="fixed">  <!--Not fixed. Change for simulation -->
+			<origin xyz="${0.2105/2} 0 0.029" rpy="1.5708 0 0"/>
+			<axis xyz="0 0 1"/>
+			<parent link="${prefix}chassis"/>
+			<child link="${prefix}passive_caster_wheel"/>
+		</joint>
     </xacro:macro>
 </robot>
