Commit message: fixed simulation

File: galax_description/urdf/galax.urdf.xacro (robot description, xacro)
@@ -1,40 +1,42 @@
 <?xml version="1.0"?>
-<robot xmlns:xacro="http://ros.org/wiki/xacro" name="galax_robot" >
+<robot xmlns:xacro="http://ros.org/wiki/xacro">
   <!-- Load the arguments -->
   <xacro:arg name="use_ros2_control" default="true"/>
   <xacro:arg name="sim_mode" default="true"/>
-  <!-- ROBOT -->
-  <!-- Add the real robot -->
-  <xacro:unless value="$(arg sim_mode)">
-    <!-- Instantiate the Pioneer3DX -->
-    <xacro:include filename="$(find galax_description)/urdf/pioneer3dx.urdf.xacro"/>
-    <xacro:pioneer3dx prefix="">
-      <origin xyz="0 0 0" rpy="0 0 0"/>
-    </xacro:pioneer3dx>
-  </xacro:unless>
-  <!-- Or the simulated robot -->
-  <xacro:if value="$(arg sim_mode)">
-    <!-- Instantiate the Pioneer3DX -->
-    <xacro:include filename="$(find galax_description)/urdf/pioneer3dx_sim.urdf.xacro"/>
-    <xacro:pioneer3dx prefix="">
-      <origin xyz="0 0 0" rpy="0 0 0"/>
-    </xacro:pioneer3dx>
-  </xacro:if>
-  <!-- CONTROLLER -->
-  <!-- Add the diffdrive controler -->
-  <xacro:unless value="$(arg sim_mode)">
-    <xacro:include filename="$(find diffdrive_arduino)/urdf/diffbot.ros2_control.xacro" />
-    <xacro:diffbot_ros2_control name="DiffBot" prefix="" device="/dev/ttyACM0" baud_rate="57600"/>
-  </xacro:unless>
-  <!-- Or the Gazebo plugin -->
-  <xacro:if value="$(arg sim_mode)">
-    <xacro:include filename="$(find galax_description)/urdf/gazebo_control.xacro"/>
-    <xacro:gazebo_control prefix=""/>
-  </xacro:if>
-  <!-- LIDAR -->
-  <!-- Mount the lidar -->
-  <xacro:include filename="$(find urg_node)/urdf/hokuyo_ust10.urdf.xacro"/>
-  <xacro:hokuyo_ust10_mount prefix="hokuyo" topic="scan" parent_link="top_plate">
-    <origin xyz="0.16 0 0" rpy="0 0 0"/>
-  </xacro:hokuyo_ust10_mount>
+  <xacro:macro name="galax_robot" params="prefix *origin">
+    <!-- ROBOT -->
+    <!-- Add the real robot -->
+    <xacro:unless value="$(arg sim_mode)">
+      <!-- Instantiate the Pioneer3DX -->
+      <xacro:include filename="$(find galax_description)/urdf/pioneer3dx.urdf.xacro"/>
+      <xacro:pioneer3dx prefix="${prefix}">
+        <origin xyz="0 0 0" rpy="0 0 0"/>
+      </xacro:pioneer3dx>
+    </xacro:unless>
+    <!-- Or the simulated robot -->
+    <xacro:if value="$(arg sim_mode)">
+      <!-- Instantiate the Pioneer3DX -->
+      <xacro:include filename="$(find galax_description)/urdf/pioneer3dx_sim.urdf.xacro"/>
+      <xacro:pioneer3dx prefix="${prefix}">
+        <origin xyz="0 0 0" rpy="0 0 0"/>
+      </xacro:pioneer3dx>
+    </xacro:if>
+    <!-- CONTROLLER -->
+    <!-- Add the diffdrive controler -->
+    <xacro:unless value="$(arg sim_mode)">
+      <xacro:include filename="$(find diffdrive_arduino)/urdf/diffbot.ros2_control.xacro" />
+      <xacro:diffbot_ros2_control name="DiffBot" prefix="${prefix}" device="/dev/ttyACM0" baud_rate="57600"/>
+    </xacro:unless>
+    <!-- Or the Gazebo plugin -->
+    <xacro:if value="$(arg sim_mode)">
+      <xacro:include filename="$(find galax_description)/urdf/gazebo_control.xacro"/>
+      <xacro:gazebo_control prefix="${prefix}"/>
+    </xacro:if>
+    <!-- LIDAR -->
+    <!-- Mount the lidar -->
+    <xacro:include filename="$(find urg_node)/urdf/hokuyo_ust10.urdf.xacro"/>
+    <xacro:hokuyo_ust10_mount prefix="hokuyo" topic="scan" parent_link="${prefix}top_plate">
+      <origin xyz="0.16 0 0" rpy="0 0 0"/>
+    </xacro:hokuyo_ust10_mount>
+  </xacro:macro>
 </robot>

File: galax_description/urdf/gazebo_control.xacro (robot description, xacro)
@@ -25,5 +25,5 @@
         <gazebo>
             <plugin name="gazebo_ros2_control" filename="libgazebo_ros2_control.so">
-                <parameters>$(find galax_description)/config/my_controllers.yaml</parameters>
+                <parameters>$(find galax_description)/config/controller_config.yaml</parameters>
 				<parameters>$(find galax_description)/config/gaz_ros2_ctl_use_sim.yaml</parameters>
             </plugin>

File: galax_description/urdf/pioneer3dx_sim.urdf.xacro (robot description, xacro)
@@ -46,5 +46,5 @@
 		</link>
 		<gazebo reference="${prefix}chassis">
-			<material>Gazebo/Red</material>
+			<material value="Gazebo/Red"/>
 		</gazebo>
 		<joint name="${prefix}chassis_joint" type="fixed">
@@ -64,5 +64,5 @@
 		</link>
 		<gazebo reference="${prefix}top_plate">
-			<material>Gazebo/Black</material>
+			<material value="Gazebo/Black"/>
 		</gazebo>
 		<joint name="${prefix}base_top_joint" type="fixed">
@@ -193,6 +193,6 @@
 		<gazebo reference="${prefix}right_wheel">
 			<material value="Gazebo/Black"/>
-            <mu1 value="10000000.0"/>
-			<mu2 value="10000000.0"/>
+			<mu1 value="10000.0"/>
+			<mu2 value="10000.0"/>
 		</gazebo>
 		<joint name="${prefix}right_wheel_joint" type="continuous">
@@ -203,4 +203,5 @@
 		</joint>
         <!-- CASTER WHEEL LINK -->
+		<!-- Swivel -->
 		<link name="${prefix}caster_swivel">
 			<visual>

Commit message: trimmed description

File: galax_description/urdf/galax.urdf.xacro (robot description, xacro)
@@ -6,20 +6,9 @@
   <xacro:macro name="galax_robot" params="prefix *origin">
     <!-- ROBOT -->
-    <!-- Add the real robot -->
-    <xacro:unless value="$(arg sim_mode)">
-      <!-- Instantiate the Pioneer3DX -->
-      <xacro:include filename="$(find galax_description)/urdf/pioneer3dx.urdf.xacro"/>
-      <xacro:pioneer3dx prefix="${prefix}">
-        <origin xyz="0 0 0" rpy="0 0 0"/>
-      </xacro:pioneer3dx>
-    </xacro:unless>
-    <!-- Or the simulated robot -->
-    <xacro:if value="$(arg sim_mode)">
-      <!-- Instantiate the Pioneer3DX -->
-      <xacro:include filename="$(find galax_description)/urdf/pioneer3dx_sim.urdf.xacro"/>
-      <xacro:pioneer3dx prefix="${prefix}">
-        <origin xyz="0 0 0" rpy="0 0 0"/>
-      </xacro:pioneer3dx>
-    </xacro:if>
+    <!-- Add the robot -->
+    <xacro:include filename="$(find galax_description)/urdf/pioneer3dx.urdf.xacro"/>
+    <xacro:pioneer3dx prefix="${prefix}">
+      <origin xyz="0 0 0" rpy="0 0 0"/>
+    </xacro:pioneer3dx>
     <!-- CONTROLLER -->
     <!-- Add the diffdrive controler -->

File: galax_description/urdf/pioneer3dx.urdf.xacro (robot description, xacro)
@@ -1,81 +1,80 @@
 <?xml version="1.0"?>
 <robot xmlns:xacro="http://www.ros.org/wiki/xacro" >
-	<xacro:include filename="$(find amr-ros-config)/urdf/materials.xacro"/>
-	<xacro:include filename="$(find amr-ros-config)/urdf/inertial_macros.xacro"/>
-	<xacro:macro name="pioneer3dx" params="prefix *origin">
-		<!-- <xacro:include filename="$(find amr-ros-config)/urdf/pioneer3dx/pioneer3dx_wheel.xacro"/> -->
-		<link name="${prefix}base_link">
-    	</link>
-		<!-- Base Link -->
+    <xacro:include filename="$(find galax_description)/urdf/materials.xacro"/>
+	<xacro:include filename="$(find galax_description)/urdf/inertial_macros.xacro"/>
+    <xacro:macro name="pioneer3dx" params="prefix *origin">
+		<!-- Chassis -->
 		<xacro:property name="chassis_length" value="0.41"/>
 		<xacro:property name="chassis_width" value="0.272"/>
 		<xacro:property name="chassis_height" value="0.172"/>
-		<link name="${prefix}real_base_link">
-			<xacro:inertial_box mass="7.0" x="${chassis_length}" y="${chassis_width}" z="${chassis_height}">
-            	<origin xyz="${-chassis_length/2} 0 ${chassis_height/2}" rpy="0 0 0"/>
-        	</xacro:inertial_box>
-			<visual>
-				<origin xyz="-0.045 0 0.148" rpy="0 0 0"/>
-				<geometry>
-					<mesh filename="file://$(find amr-ros-config)/meshes/p3dx_meshes/chassis.stl"/>
-				</geometry>
-				<material name="ChassisRed"/>
-			</visual>
-			<!-- <collision>
-				<origin xyz="-0.045 0 0.148" rpy="0 0 0"/>
-				<geometry>
-					<mesh filename="file://$(find amr-ros-config)/meshes/p3dx_meshes/chassis.stl"/>
-				</geometry>
-			</collision> -->
-		</link>
-		<gazebo reference="${prefix}real_base_link">
-			<material>Gazebo/Red</material>
-		</gazebo>
-		<joint name="${prefix}real_base_link_joint" type="fixed">
-			<origin xyz="0 0 0" rpy="0 0 0"/>
-			<parent link="${prefix}base_link"/>
-			<child link="${prefix}real_base_link"/>
-		</joint>
+		<xacro:property name="chassis_mass" value="5.0"/>
 		<!-- Top Plate -->
 		<xacro:property name="top_plate_length" value="0.41"/>
 		<xacro:property name="top_plate_width" value="0.272"/>
 		<xacro:property name="top_plate_height" value="0.0052"/>
+		<xacro:property name="top_plate_mass" value="0.01"/>
+		<!-- Wheels -->
+		<xacro:property name="wheel_radius" value="0.09"/>
+		<xacro:property name="wheel_thickness" value="0.04"/>
+		<xacro:property name="wheel_mass" value="0.5"/>
+		<!-- Caster wheel -->
+		<xacro:property name="caster_wheel_radius" value="0.0375"/>
+		<xacro:property name="caster_wheel_thickness" value="0.01"/>
+		<xacro:property name="caster_wheel_mass" value="0.01"/>
+        <!-- BASE LINK -->
+        <link name="${prefix}base_link">
+        </link>
+        <!-- CHASSIS LINK -->
+		<link name="${prefix}chassis">
+			<collision>
+				<origin xyz="0 0 ${chassis_height/2}"/>
+				<geometry>
+					<!-- <box size="0 0 0"/> -->
+					<box size="${chassis_length/4} ${chassis_width/4} ${chassis_height/4}"/>
+				</geometry>
+			</collision>
+			<visual>
+				<origin xyz="-0.045 0 0.148" rpy="0 0 0"/>
+				<geometry>
+					<mesh filename="file://$(find galax_description)/meshes/chassis.stl"/>
+				</geometry>
+				<material name="ChassisRed"/>
+			</visual>
+			<xacro:inertial_box mass="${chassis_mass}" x="${chassis_length}" y="${chassis_width}" z="${chassis_height}">
+            	<origin xyz="0 0 ${chassis_height/2}" rpy="0 0 0"/>
+        	</xacro:inertial_box>
+		</link>
+		<gazebo reference="${prefix}chassis">
+			<material value="Gazebo/Red"/>
+		</gazebo>
+		<joint name="${prefix}chassis_joint" type="fixed">
+			<origin xyz="0 0 0" rpy="0 0 0"/>
+			<parent link="${prefix}base_link"/>
+			<child link="${prefix}chassis"/>
+		</joint>
+		<!-- Top Plate -->
 		<link name="${prefix}top_plate">
-			<xacro:inertial_box mass="0.1" x="${top_plate_length}" y="${top_plate_width}" z="${top_plate_height}">
-            	<origin xyz="${chassis_length/2} 0 ${chassis_height/2}" rpy="0 0 0"/>
-        	</xacro:inertial_box>
-			<visual>
-				<origin xyz="0 0 0" rpy="0 0 0"/>
-				<geometry>
-					<mesh filename="file://$(find amr-ros-config)/meshes/p3dx_meshes/top.stl"/>
+			<visual>
+				<origin xyz="0 0 0" rpy="0 0 0"/>
+				<geometry>
+					<mesh filename="file://$(find galax_description)/meshes/top.stl"/>
 				</geometry>
 				<material name="TopBlack"/>
 			</visual>
-			<collision>
-				<origin xyz="0 0 0" rpy="0 0 0"/>
-				<geometry>
-					<mesh filename="file://$(find amr-ros-config)/meshes/p3dx_meshes/top.stl"/>
-				</geometry>
-			</collision>
 		</link>
 		<gazebo reference="${prefix}top_plate">
-			<material>Gazebo/Black</material>
+			<material value="Gazebo/Black"/>
 		</gazebo>
 		<joint name="${prefix}base_top_joint" type="fixed">
 			<origin xyz="-0.045 0 0.234" rpy="0 0 0"/>
-			<parent link="${prefix}real_base_link"/>
+			<parent link="${prefix}chassis"/>
 			<child link="${prefix}top_plate"/>
 		</joint>
 		<!-- Front Sonar -->
 		<link name="${prefix}front_sonar">
-			<inertial>
-				<mass value="0.0001"/>
-				<origin xyz="0 0 0"/>
-				<inertia ixx="1" ixy="0" ixz="0" iyy="1" iyz="0" izz="1"/>
-			</inertial>
-			<visual>
-				<origin xyz="0 0 0" rpy="0 0 0"/>
-				<geometry>
-					<mesh filename="file://$(find amr-ros-config)/meshes/p3dx_meshes/front_sonar.stl"/>
+			<visual>
+				<origin xyz="0 0 0" rpy="0 0 0"/>
+				<geometry>
+					<mesh filename="file://$(find galax_description)/meshes/front_sonar.stl"/>
 				</geometry>
 				<material name="SonarYellow"/>
@@ -87,84 +86,149 @@
 		<joint name="${prefix}base_front_joint" type="fixed">
 			<origin xyz="-0.198 0 0.208" rpy="0 0 0"/>
-			<parent link="${prefix}real_base_link"/>
+			<parent link="${prefix}chassis"/>
 			<child link="${prefix}front_sonar"/>
 		</joint>
 		<!-- Back Sonar -->
+		<link name="${prefix}back_sonar">
+			<visual>
+				<origin xyz="0 0 0" rpy="0 0 0"/>
+				<geometry>
+					<mesh filename="file://$(find galax_description)/meshes/back_sonar.stl"/>
+				</geometry>
+				<material name="SonarYellow"/>
+			</visual>
+		</link>
+		<gazebo reference="${prefix}back_sonar">
+			<material value="Gazebo/Yellow"/>
+		</gazebo>
 		<joint name="${prefix}base_back_joint" type="fixed">
 			<origin xyz="0.109 0 0.209" rpy="0 0 0"/>
-			<parent link="${prefix}real_base_link"/>
+			<parent link="${prefix}chassis"/>
 			<child link="${prefix}back_sonar"/>
 		</joint>
-		<link name="${prefix}back_sonar">
-			<inertial>
-				<mass value="0.0001"/>
-				<origin xyz="0 0 0"/>
-				<inertia ixx="1" ixy="0" ixz="0" iyy="1" iyz="0" izz="1"/>
-			</inertial>
-			<visual>
-				<origin xyz="0 0 0" rpy="0 0 0"/>
-				<geometry>
-					<mesh filename="file://$(find amr-ros-config)/meshes/p3dx_meshes/back_sonar.stl"/>
-				</geometry>
-				<material name="SonarYellow"/>
-			</visual>
-		</link>
-		<gazebo reference="${prefix}back_sonar">
-			<material value="Gazebo/Yellow"/>
-		</gazebo>
-		<!-- Caster Swivel -->
-		<joint name="${prefix}base_caster_swivel_joint" type="fixed"> <!--Not fixed. Change for simulation -->
-			<origin xyz="-0.185 0 0.055" rpy="0 0 0"/>
-			<axis xyz="0 0 1"/>
-			<parent link="${prefix}real_base_link"/>
-			<child link="${prefix}caster_swivel"/>
-			<limit effort="10000.0" lower="-100000" upper="100000" velocity="100000"/>
-    		<!-- <dynamics damping="0.001" friction="0.0001"/> -->
-		</joint>
-		<passive_joint name="${prefix}base_caster_swivel_joint"/> <!--Not working -->
+        <!-- LEFT WHEEL LINK -->
+		<link name="${prefix}left_hub">
+			<visual>
+				<origin xyz="0 0 0" rpy="${-3.1415927/2.0} 0 0"/>
+				<geometry>
+					<cylinder radius="0.09" length="0.01"/>
+				</geometry>
+				<material name="HubcapYellow"/>
+			</visual>
+		</link>
+		<gazebo reference="${prefix}left_hub">
+			<material value="Gazebo/Yellow"/>
+		</gazebo>
+		<joint name="${prefix}left_hub_joint" type="fixed">
+			<origin xyz="0 0.15 0.08" rpy="0 0 0"/>
+			<parent link="${prefix}chassis"/>
+			<child link="${prefix}left_hub"/>
+			<axis xyz="0 1 0"/>
+		</joint>
+		<link name="${prefix}left_wheel">
+			<collision>
+				<origin xyz="0 0 0" rpy="0 0 0"/>
+				<geometry>
+					<sphere radius="${wheel_radius}"/>
+				</geometry>
+			</collision>
+			<visual>
+				<origin xyz="0 0 0" rpy="1.5708 0 0"/>
+				<geometry>
+					<mesh filename="file://$(find galax_description)/meshes/left_wheel.stl"/>
+				</geometry>
+				<material name="WheelBlack"/>
+			</visual>
+			<xacro:inertial_cylinder mass="${wheel_mass}" length="${wheel_thickness}" radius="${wheel_radius}">
+				<origin xyz="0 0 0" rpy="0 0 0"/>
+			</xacro:inertial_cylinder>
+		</link>
+		<gazebo reference="${prefix}left_wheel">
+			<material value="Gazebo/Black"/>
+            <mu1 value="10000.0"/>
+			<mu2 value="10000.0"/>
+		</gazebo>
+		<joint name="${prefix}left_wheel_joint" type="continuous">
+			<origin xyz="0 0.15 0.08" rpy="-1.5708 0 0"/>
+			<axis xyz="0 0 1"/>
+			<parent link="${prefix}chassis"/>
+			<child link="${prefix}left_wheel"/>
+		</joint>
+        <!-- RIGHT WHEEL LINK -->
+		<link name="${prefix}right_hub">
+			<visual>
+				<origin xyz="0 0 0" rpy="${3.1415927/2.0} 0 0"/>
+				<geometry>
+					<cylinder radius="0.09" length="0.01"/>
+				</geometry>
+				<material name="HubcapYellow"/>
+			</visual>
+		</link>
+		<gazebo reference="${prefix}right_hub">
+			<material value="Gazebo/Yellow"/>
+		</gazebo>
+		<joint name="${prefix}right_hub_joint" type="fixed">
+			<origin xyz="0 -0.15 0.08" rpy="0 0 0"/>
+			<parent link="${prefix}chassis"/>
+			<child link="${prefix}right_hub"/>
+		</joint>
+		<link name="${prefix}right_wheel">
+			<collision>
+				<origin xyz="0 0 0" rpy="0 0 0"/>
+				<geometry>
+					<sphere radius="${wheel_radius}"/>
+				</geometry>
+			</collision>
+			<visual>
+				<origin xyz="0 0 0" rpy="-1.5708 0 0"/>
+				<geometry>
+					<mesh filename="file://$(find galax_description)/meshes/right_wheel.stl"/>
+				</geometry>
+				<material name="WheelBlack"/>
+			</visual>
+			<xacro:inertial_cylinder mass="${wheel_mass}" length="${wheel_thickness}" radius="${wheel_radius}">
+				<origin xyz="0 0 0" rpy="0 0 0"/>
+			</xacro:inertial_cylinder>
+		</link>
+		<gazebo reference="${prefix}right_wheel">
+			<material value="Gazebo/Black"/>
+			<mu1 value="10000.0"/>
+			<mu2 value="10000.0"/>
+		</gazebo>
+		<joint name="${prefix}right_wheel_joint" type="continuous">
+			<origin xyz="0 -0.15 0.08" rpy="1.5708 0 0"/>
+			<axis xyz="0 0 -1"/>
+			<parent link="${prefix}chassis"/>
+			<child link="${prefix}right_wheel"/>
+		</joint>
+        <!-- CASTER WHEEL LINK -->
+		<!-- Swivel -->
 		<link name="${prefix}caster_swivel">
-			<inertial>
-				<mass value="0.01"/>
-				<origin xyz="0 0 0"/>
-				<inertia ixx="0.01" ixy="0" ixz="0" iyy="0.01" iyz="0" izz="0.01"/>
-			</inertial>
-			<visual>
-				<origin xyz="0 0 0" rpy="0 0 0"/>
-				<geometry>
-					<mesh filename="file://$(find amr-ros-config)/meshes/p3dx_meshes/caster_swivel.stl"/>
+			<visual>
+				<origin xyz="0 0 0" rpy="0 0 0"/>
+				<geometry>
+					<mesh filename="file://$(find galax_description)/meshes/caster_swivel.stl"/>
 				</geometry>
 				<material name="ChassisGrey"/>
 			</visual>
-			<!-- <collision>
-				<origin xyz="0 0 0" rpy="0 0 0"/>
-				<geometry>
-					<mesh filename="file://$(find amr-ros-config)/meshes/p3dx_meshes/caster_swivel.stl"/>
-				</geometry>
-			</collision> -->
 		</link>
 		<gazebo reference="${prefix}caster_swivel">
 			<material value="Gazebo/Grey"/>
 		</gazebo>
-		<!-- Center Wheel + Hubcap -->
+		<joint name="${prefix}base_caster_swivel_joint" type="fixed"> <!--Not fixed. Change for simulation -->
+			<origin xyz="-0.185 0 0.045" rpy="0 0 0"/>
+			<axis xyz="0 0 1"/>
+			<parent link="${prefix}chassis"/>
+			<child link="${prefix}caster_swivel"/>
+		</joint>
+		<!-- Hubcap -->
 		<link name="${prefix}caster_hubcap">
-			<inertial>
-				<mass value="0.01"/>
-				<origin xyz="0 0 0"/>
-				<inertia ixx="0.012411765597" ixy="-0.000711733678" ixz="0.00050272983"
-							iyy="0.015218160428" iyz="-0.000004273467" izz="0.011763977943"/>
-			</inertial>
 			<visual>
 				<origin xyz="0 0 0" rpy="${1.5708} 0 0"/>
 				<geometry>
-					<mesh filename="file://$(find amr-ros-config)/meshes/p3dx_meshes/caster_hubcap.stl"/>
+					<mesh filename="file://$(find galax_description)/meshes/caster_hubcap.stl"/>
 				</geometry>
 				<material name="ChassisGrey"/>
 			</visual>
-			<!-- <collision>
-				<origin xyz="0 0 0" rpy="0 0 0"/>
-				<geometry>
-					<mesh filename="file://$(find amr-ros-config)/meshes/p3dx_meshes/caster_hubcap.stl"/>
-				</geometry>
-			</collision> -->
 		</link>
 		<gazebo reference="${prefix}caster_hubcap">
@@ -176,170 +240,55 @@
 			<parent link="${prefix}caster_swivel"/>
 			<child link="${prefix}caster_hubcap"/>
-			<limit effort="10000.0" lower="-100000" upper="100000" velocity="100000"/>
-    		<!-- <dynamics damping="0.001" friction="0.0001"/> -->
 		</joint>
 		<!-- Caster Wheel -->
 		<link name="${prefix}caster_wheel">
-			<xacro:inertial_cylinder mass="0.2" length="0.01" radius="0.0375">
-				<origin xyz="0 0 0" rpy="0 0 0"/>
+			<collision>
+				<origin xyz="0 0 0" rpy="0 0 0"/>
+				<geometry>
+					<sphere radius="${caster_wheel_radius}"/>
+				</geometry>
+			</collision>
+			<visual>
+				<origin xyz="0 0 0" rpy="0 0 0"/>
+				<geometry>
+					<cylinder radius="${caster_wheel_radius}" length="${caster_wheel_thickness}"/>
+				</geometry>
+				<material name="WheelBlack"/>
+			</visual>
+			<xacro:inertial_cylinder mass="${caster_wheel_mass}" length="${caster_wheel_thickness}" radius="${caster_wheel_radius}">
+				<origin xyz="0.185 0 0" rpy="0 0 0"/>
 			</xacro:inertial_cylinder>
-			<visual>
-				<origin xyz="0 0 0" rpy="0 0 0"/>
-				<geometry>
-					<cylinder radius="0.0375" length="0.01"/>
-				</geometry>
-				<material name="WheelBlack"/>
-			</visual>
-			<collision>
-				<origin xyz="0 0 0" rpy="0 0 0"/>
-				<geometry>
-					<cylinder radius="0.0375" length="0.01"/>
-				</geometry>
-			</collision>
-			<dynamics damping="10.0" friction="0"/>
 		</link>
 		<gazebo reference="${prefix}caster_wheel">
-			<material value="Gazebo/Black"/>
+			<material value="Gazebo/White"/>
+			<mu1 value="0.00001"/>
+			<mu2 value="0.00001"/>
 		</gazebo>
 		<joint name="${prefix}caster_wheel_joint" type="fixed">  <!--Not fixed. Change for simulation -->
-			<origin xyz="-0.0035 0 -0.001" rpy="0 0 0"/>
-			<axis xyz="0 0 1"/>
-			<parent link="${prefix}caster_hubcap"/>
+			<origin xyz="-0.2105 0 0.029" rpy="1.5708 0 0"/>
+			<axis xyz="0 0 1"/>
+			<parent link="${prefix}chassis"/>
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